Commit message: remove_type_in_base_link

File: my_robot6.xacro (robot description, xacro)
@@ -13,5 +13,5 @@
     <xacro:property name="sphere_radius" value="0.3" />
     <xacro:include filename="/home/ranzant197/material_color.xacro" />
-    <link name="base_link" type="fixed">
+    <link name="base_link">
         <visual>
             <geometry>
